File: Data/board3.brd (EAGLE design)
At the start: 70 x 67.5 mm, 78 parts, among them Q1 16MHz, U1 ACPL224, U10 VO1400, U11 VO1400, U12 VO1400, U13 VO1400, U14 VO1400, U15 VO1400, U16 VO1400, U17 VO1400, U18 LH1522AAC, U19 MCP1703T-3302E/MB, U2 ACPL224, U20 MAX3232CSE, U21 PIC18F46K22-I/PT, U3 ACPL224, U4 ACPL224, U5 ACPL224, U6 ACPL224, U7 ACPL224, U8 VO1400, U9 VO1400

Commit message: Commit final del dia
Signed-off-by: Rafael Serrano <rsr.private@gmail.com>
Parts:
- C14, C16: device rcl:SMC_A -> smd-parts:C-SMC-A
- L1: device rcl-2:L0805 -> smd-parts:L-0805
- LED1: device led:CHIPLED_0805 -> smd-parts:D-LED-0805
- turned LED1 to 270 degrees
Connections:
- net GND: now also C14.2, C16.2, LED1.1; no longer C14.-, C16.-, LED1.C
- net N$22: now also LED1.2; no longer LED1.A
- net VCC: now also C14.1, C16.1; no longer C14.+, C16.+

Commit message: Commit final del dia
Signed-off-by: Rafael Serrano <rsr.private@gmail.com>
Connections:
- net GND: now also LED1.C; no longer LED1.1
- net N$22: now also LED1.A; no longer LED1.2
Changed lines of the file:
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@@
 </autorouter>
 <elements>
-<element name="U$3" library="holes" package="3,6" value="" x="65.5" y="4.5" locked="yes"/>
+<element name="U$3" library="holes" package="3,6" value="" x="65.5" y="4.5" locked="yes">
+<attribute name="PARTLIST-IGNORE" value="" x="65.5" y="4.5" size="1.778" layer="27" display="off"/>
+</element>
 <element name="JP5" library="pinhead200" package="1X05-2MM" value="ICSP" x="39.25" y="8.5" locked="yes" smashed="yes">
 <attribute name="NAME" x="38.75" y="10" size="1.016" layer="25"/>
@@
 <attribute name="REFERENCE" value="DF13-4P-1.25H(20)" x="6.5" y="40.75" size="1.778" layer="27" rot="R90" display="off"/>
 </element>
-<element name="U$6" library="holes" package="3,6" value="" x="65.5" y="63" locked="yes"/>
+<element name="U$6" library="holes" package="3,6" value="" x="65.5" y="63" locked="yes">
+<attribute name="PARTLIST-IGNORE" value="" x="65.5" y="63" size="1.778" layer="27" display="off"/>
+</element>
 <element name="C7" library="smd-parts" package="C-0805" value="100n" x="38" y="27.75" locked="yes" smashed="yes" rot="R270">
 <attribute name="NAME" x="38" y="29.75" size="1.016" layer="25" align="bottom-center"/>
@@
 <attribute name="MANUFACTURER" value="Vishay" x="65.625" y="43" size="1.778" layer="27" rot="R270" display="off"/>
 </element>
-<element name="U$9" library="holes" package="3,6" value="" x="4.5" y="63" locked="yes"/>
-<element name="U$10" library="holes" package="3,6" value="" x="4.5" y="4.5" locked="yes"/>
+<element name="U$9" library="holes" package="3,6" value="" x="4.5" y="63" locked="yes">
+<attribute name="PARTLIST-IGNORE" value="" x="4.5" y="63" size="1.778" layer="27" display="off"/>
+</element>
+<element name="U$10" library="holes" package="3,6" value="" x="4.5" y="4.5" locked="yes">
+<attribute name="PARTLIST-IGNORE" value="" x="4.5" y="4.5" size="1.778" layer="27" display="off"/>
+</element>
 <element name="JP3" library="hirose-df13" package="1X5-SMD-90-E" value="DF13-1X5-SMD-90-E" x="6.5" y="14.25" locked="yes" smashed="yes" rot="R90">
 <attribute name="NAME" x="5.25" y="9.5" size="1" layer="25"/>
@@
 <contactref element="C16" pad="2"/>
 <contactref element="C17" pad="1"/>
-<contactref element="LED1" pad="1"/>
+<contactref element="LED1" pad="C"/>
 <polygon width="0.15" layer="1">
 <vertex x="0.25" y="52.5"/>
@@
 <signal name="N$22">
 <contactref element="R19" pad="1"/>
-<contactref element="LED1" pad="2"/>
+<contactref element="LED1" pad="A"/>
 <wire x1="23.75" y1="8.7" x2="25.65" y2="8.7" width="0.2" layer="1"/>
 <wire x1="25.65" y1="8.7" x2="25.75" y2="8.8" width="0.2" layer="1"/>

Commit message: Commit final del dia
Signed-off-by: Rafael Serrano <rsr.private@gmail.com>
Parts:
- removed JP1: DF11-18DP-2DSA, hirose-df11:DF11-18DP-2DSA
- removed JP2: DF11-16DP-2DSA, hirose-df11:DF11-16DP-2DSA
- removed JP7: DF13-1X4-SMD-90-E, hirose-df13:1X4-SMD-90-E
- removed R20, R21: 270, smd-parts:R-0805
- removed R22, R23, R7, R8: 10K, smd-parts:R-0805
- removed U19: MCP1703T-3302E/MB, microchip-analog:SOT89
- removed U20: MAX3232CSE, maxim:SO16
- removed U21: PIC18F46K22-I/PT, microchip-pic:TQFP44
- added JP8: DF13-1X4-SMD-90-E, hirose-df13:1X4-SMD-90-E
- added X1, X2: 2514-5, con-3m:PAK100/2500-5-14
- C1, C10, C11, C12, C13, C15, C17, C2, C3, C4, C5, C6, C7, C8, C9: device smd-parts:C-0805 -> rcl:C0805
- C14, C16: device smd-parts:C-SMC-A -> rcl:SMC_A
- L1: device smd-parts:L-0805 -> rcl-2:L0805
- LED1: device smd-parts:D-LED-0805 -> led:CHIPLED_1206
- R1, R10, R11, R12, R13, R14, R15, R16, R17, R18, R19, R2, R3, R4, R5, R6, R9: device smd-parts:R-0805 -> rcl:R0805
- U$1: device logo:CE_7.3MM -> logo:CE-4MM
- U10: value VO1400 -> PIC18F46K22-I/PT; device optoacopladores:SOP04 -> microchip-pic:TQFP44
- U11: value VO1400 -> MAX3232CSE; device optoacopladores:SOP04 -> maxim:SO16
- U12: value VO1400 -> ACPL224; device optoacopladores:SOP04 -> optoacopladores:SO08
- U18: value LH1522AAC -> VO1400; device optoacopladores:DIL8-SMD -> optoacopladores:SOP04
- U5, U6, U7: value ACPL224 -> VO1400; device optoacopladores:SO08 -> optoacopladores:SOP04
- U9: value VO1400 -> MCP17033302I/MB; device optoacopladores:SOP04 -> microchip-analog:SOT89
- moved U11 40.8 mm to (13.5, 15.0), turned to 90 degrees
- moved U$2 37.9 mm to (11.2, 27.8)
- moved U$1 35.1 mm to (44.5, 28.5)
- moved D2 34.7 mm to (67.0, 39.0), turned to 0 degrees
- moved R1 30.9 mm to (67.5, 35.5), turned to 90 degrees
- moved C13 28.5 mm to (62.0, 39.0), turned to 180 degrees
- moved U10 27.7 mm to (34.0, 18.5), turned to 90 degrees
- moved C12 27.7 mm to (62.0, 32.0), turned to 0 degrees
- moved L1 24.9 mm to (67.5, 32.0), turned to 180 degrees
- moved U12 24.4 mm to (27.0, 47.5), turned to 180 degrees
- moved U14 21.3 mm to (49.5, 47.0), flipped to the bottom, turned to 0 degrees
- moved U9 19.8 mm to (62.5, 35.5)
- moved U13 18.4 mm to (49.5, 47.0), turned to 0 degrees
- moved U5 16.1 mm to (39.5, 47.0), turned to 0 degrees
- moved R15 15.5 mm to (54.5, 39.5), turned to 90 degrees
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Connections:
- removed net I10: JP1.13, U6.2
- removed net I11: JP1.14, U6.4
- removed net I12: JP1.15, U7.2
- removed net I13A: JP1.17, U7.3
- removed net I13B: JP1.18, U7.4
- removed net IC0: JP1.5, U1.1, U1.3, U2.1, U2.3
- removed net IC1: JP1.10, U3.1, U3.3, U4.1, U4.3
- removed net IC2: JP1.16, U5.1, U5.3, U6.1, U6.3, U7.1
- removed net IN10: R7.1, U21.41, U6.8
- removed net IN11: R8.1, U21.2, U6.6
- removed net IN12: R22.1, U21.42, U7.8
- removed net IN13: R23.1, U21.37, U7.6
- removed net N$48: R21.2, U18.3
- removed net N$9: R20.2, U18.1
- removed net O10A: JP2.13, U18.8
- removed net O10B: JP2.14, U18.7
- removed net O11A: JP2.15, U18.6
- removed net O11B: JP2.16, U18.5
- removed net OC0: JP2.6, U10.3, U11.3, U12.3, U8.3, U9.3
- removed net OC1: JP2.12, U13.3, U14.3, U15.3, U16.3, U17.3
- removed net OUT10: R20.1, U21.40
- removed net OUT11: R21.1, U21.27
- new net I-COM0: U1.1, U1.3, U2.1, X1.11
- new net I-COM1: U2.3, U3.1, U3.3, X1.12
- new net I-COM2: U4.1, U4.3, X1.13
- new net I-COM3: U12.1, U12.3, X1.14
- new net O-COM0: U5.3, U6.3, U7.3, X2.11
- new net O-COM1: U13.3, U14.3, U8.3, X2.12
- new net O-COM2: U15.3, U16.3, X2.13
- new net O-COM3: U17.3, U18.3, X2.14
- net GND: now also C14.-, C16.-, JP8.4, U10.29, U10.6, U11.15, U12.5, U12.7, U5.2, U6.2, U7.2, U9.1; no longer C14.2, C16.2, JP7.4, U10.2, U11.2, U12.2, U18.4, U19.1, U20.15, U21.29, U21.6, U5.5, U5.7, U6.5, U6.7, U7.5, U7.7, U9.2
- net I0: now also X1.1; no longer JP1.1
- net I1: now also X1.2; no longer JP1.2
- net I2: now also X1.3; no longer JP1.3
- net I3: now also X1.4; no longer JP1.4
- net I4: now also X1.5; no longer JP1.6
- net I5: now also X1.6; no longer JP1.7
- net I6: now also X1.7; no longer JP1.8
- net I7: now also X1.8; no longer JP1.9
- net I8: now also U12.2, X1.9; no longer JP1.11, U5.2
- net I9: now also U12.4, X1.10; no longer JP1.12, U5.4
- net IN0: now also U10.9; no longer U21.9
- net IN1: now also U10.8; no longer U21.8
- net IN2: now also U10.11; no longer U21.11
- net IN3: now also U10.10; no longer U21.10
- net IN4: now also U10.15; no longer U21.15
- net IN5: now also U10.14; no longer U21.14
- net IN6/PGD: now also U10.17; no longer U21.17
- net IN7/PGC: now also U10.16; no longer U21.16
- net IN8: now also R5.1, U10.25, U12.8; no longer R2.1, U21.25, U5.8
- net IN9: now also R2.1, U10.26, U12.6; no longer R5.1, U21.26, U5.6
- net LED: now also U10.3; no longer U21.3
- net N$1: now also U17.1; no longer U16.1
- net N$13: now also U11.7; no longer U20.7
- net N$14: now also U11.13; no longer U20.13
- net N$15: now also U11.8; no longer U20.8
- net N$16: now also U11.1; no longer U20.1
- net N$17: now also U5.1; no longer U8.1
- net N$18: now also U6.1; no longer U9.1
- net N$25: now also U7.1; no longer U10.1
- net N$26: now also U8.1; no longer U11.1
- net N$29: now also U11.3; no longer U20.3
- net N$30: now also U11.4; no longer U20.4
- net N$33: now also U11.5; no longer U20.5
- net N$34: now also U11.2; no longer U20.2
- net N$35: now also U11.6; no longer U20.6
- net N$36: now also U10.31; no longer U21.31
- net N$4: now also U11.14; no longer U20.14
- net N$5: now also U9.2, U9.2@1; no longer U19.2, U19.2@1
- net N$51: now also U15.1; no longer U14.1
- net N$52: now also U13.1; no longer U12.1
- net N$53: now also U14.1; no longer U13.1
- net N$54: now also U16.1; no longer U15.1
- net N$6: now also U18.1; no longer U17.1
- net N$8: now also U10.30; no longer U21.30
- net O0: now also U5.4, X2.1; no longer JP2.1, U8.4
- net O1: now also U6.4, X2.2; no longer JP2.2, U9.4
- net O2: now also U7.4, X2.3; no longer JP2.3, U10.4
- net O3: now also U8.4, X2.4; no longer JP2.4, U11.4
- net O4: now also U13.4, X2.5; no longer JP2.5, U12.4
- net O5: now also U14.4, X2.6; no longer JP2.7, U13.4
- net O6: now also U15.4, X2.7; no longer JP2.8, U14.4
- net O7: now also U16.4, X2.8; no longer JP2.9, U15.4
- net O8: now also U17.4, X2.9; no longer JP2.10, U16.4
- net O9: now also U18.4, X2.10; no longer JP2.11, U17.4
- net OUT0: now also U10.24; no longer U21.24
- net OUT1: now also U10.23; no longer U21.23
- net OUT2: now also U10.20; no longer U21.22
- net OUT3: now also U10.22; no longer U21.21
- net OUT4: now also U10.21; no longer U21.20
- net OUT5: now also U10.19; no longer U21.19
- net OUT6: now also U10.35; no longer U21.35
- net OUT7: now also U10.37; no longer U21.43
- net OUT8: now also U10.36; no longer U21.36
- net OUT9: now also U10.32; no longer U21.32
- net RX1: now also U10.1, U11.12; no longer U20.12, U21.1
- net RX2: now also U10.5, U11.9; no longer U20.9, U21.5
- net SCL2: now also JP8.2, U10.38; no longer JP7.2, U21.38
- net SDA2: now also JP8.3, U10.39; no longer JP7.3, U21.39
- net TX1: now also U10.44, U11.11; no longer U20.11, U21.44
- net TX2: now also U10.4, U11.10; no longer U20.10, U21.4
- net VCC: now also C14.+, C16.+, JP8.1, U10.28, U10.7, U11.16, U9.3; no longer C14.1, C16.1, JP7.1, R22.2, R23.2, R7.2, R8.2, U19.3, U20.16, U21.28, U21.7
- net VPP: now also U10.18; no longer U21.18
Routing:
- net OUT10: track 71.4 -> 0.00 mm, vias 2 -> 0
- net OUT11: track 68.3 -> 0.00 mm, vias 2 -> 0
- net IN12: track 61.0 -> 0.00 mm, vias 2 -> 0
- net IN11: track 53.0 -> 0.00 mm, vias 2 -> 0
- net IN13: track 52.0 -> 0.00 mm, vias 2 -> 0
- net OC1: track 48.2 -> 0.00 mm, vias 1 -> 0
- net IN10: track 46.2 -> 0.00 mm, vias 2 -> 0
- net O-COM1: track 0.00 -> 41.3 mm, vias 0 -> 1
- net I-COM1: track 0.00 -> 39.8 mm, vias 0 -> 3
- net OC0: track 36.9 -> 0.00 mm, vias 1 -> 0
- net I-COM0: track 0.00 -> 34.7 mm, vias 0 -> 3
- net IC2: track 30.5 -> 0.00 mm
- net O6: track 39.1 -> 8.95 mm
- net IC0: track 29.8 -> 0.00 mm
- net O4: track 35.9 -> 7.03 mm, vias 0 -> 1
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Other:
- board text added: "MD-CPU04C-v1.1"
- board text removed: "MD-CPU04D-v1.1"
