File: Data/kicad_demo.kicad_pcb (KiCad board)
At the start: 2 copper layers, 109 x 62.5 mm, 88 parts, among them U1 MCP1703A-3302_SOT89, U2 24LC1025, U3 MCP7940N-xST, U4 MCP9804_MSOP, U5 STCS05, U6 PIC32MX4H_PT, U7 MAX31911, U8 NCV7240, Y1 CM7V-T1A, Y2 ABM3B

Commit message: Revisions cosmetiques
Signed-off-by: Rafael Serrano <rsr.openware@gmail.com>
Parts:
- added REF**: x, proves:x, F.Cu at (119.6, 56.6)
